Commit message: robocon2027_world

File: src/robocon2027_description/urdf/tr.xacro (robot description, xacro)
@@ -89,42 +89,10 @@
 x="-${wheel_x}"
 y="-${wheel_y}"/>
-<ros2_control name="TRSystem" type="system">
-<hardware>
-<plugin>gz_ros2_control/GazeboSimSystem</plugin>
-</hardware>
-<joint name="front_left_wheel_joint">
-<command_interface name="velocity"/>
-<state_interface name="position"/>
-<state_interface name="velocity"/>
-</joint>
-<joint name="front_right_wheel_joint">
-<command_interface name="velocity"/>
-<state_interface name="position"/>
-<state_interface name="velocity"/>
-</joint>
-<joint name="rear_left_wheel_joint">
-<command_interface name="velocity"/>
-<state_interface name="position"/>
-<state_interface name="velocity"/>
-</joint>
-<joint name="rear_right_wheel_joint">
-<command_interface name="velocity"/>
-<state_interface name="position"/>
-<state_interface name="velocity"/>
-</joint>
-</ros2_control>
 <gazebo>
-<plugin
-filename="libgz_ros2_control-system.so"
-name="gz_ros2_control::GazeboSimROS2ControlPlugin">
-<parameters>
-$(find robocon2027_description)/config/tr_controllers.yaml
-</parameters>
-</plugin>
-</gazebo>
-<gazebo>
-<plugin
-filename="gz-sim-diff-drive-system"
-name="gz::sim::systems::DiffDrive">
+<plugin filename="libgazebo_ros_diff_drive.so" name="gazebo_ros_diff_drive">
+<ros>
+<remapping>cmd_vel:=/cmd_vel</remapping>
+</ros>
+<num_wheel_pairs>2</num_wheel_pairs>
 <left_joint>front_left_wheel_joint</left_joint>
 <left_joint>rear_left_wheel_joint</left_joint>
@@ -132,14 +100,10 @@
 <right_joint>rear_right_wheel_joint</right_joint>
 <wheel_separation>0.50</wheel_separation>
-<wheel_radius>0.075</wheel_radius>
+<wheel_diameter>0.15</wheel_diameter>
+<robot_base_frame>tr/base_link</robot_base_frame>
+<odometry_frame>tr/odom</odometry_frame>
+<publish_odom>true</publish_odom>
+<publish_odom_tf>true</publish_odom_tf>
 <odom_publish_frequency>50</odom_publish_frequency>
-<max_linear_acceleration>1.0</max_linear_acceleration>
-<min_linear_acceleration>-1.0</min_linear_acceleration>
-<max_angular_acceleration>2.0</max_angular_acceleration>
-<min_angular_acceleration>-2.0</min_angular_acceleration>
-<max_linear_velocity>1.0</max_linear_velocity>
-<min_linear_velocity>-1.0</min_linear_velocity>
-<max_angular_velocity>2.0</max_angular_velocity>
-<min_angular_velocity>-2.0</min_angular_velocity>
 </plugin>
 </gazebo>
@@ -165,7 +129,5 @@
 </joint>
 <gazebo reference="lidar_link">
-<sensor name="lidar" type="gpu_lidar">
-<topic>scan</topic>
-<frame_id>lidar_link</frame_id>
+<sensor name="lidar" type="ray">
 <update_rate>10</update_rate>
 <lidar>
@@ -191,4 +153,11 @@
 </lidar>
 <visualize>true</visualize>
+<plugin name="gazebo_ros_ray_sensor" filename="libgazebo_ros_ray_sensor.so">
+<ros>
+<remapping>~/out:=/scan</remapping>
+</ros>
+<output_type>sensor_msgs/LaserScan</output_type>
+<frame_name>tr/lidar_link</frame_name>
+</plugin>
 </sensor>
 </gazebo>
